File: PCB/PCB.kicad_sch (KiCad schematic)
At the start: 9 parts

Commit message: Pcb para imprimir
Parts:
- U1: renamed from U?; footprint (none) -> DOIT_ESP32:DOIT_ESP32_Devkit_mirko
- U2: renamed from U?; footprint (none) -> Stepdown:Step down lm
- gave numbers to parts that had none: 7
Other:
- moved on the sheet: J1
Changed lines of the file:
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@@
 	(generator_version "8.0")
 	(paper "A4")
+	(wire
+		(pts
+			(xy 54.61 114.3) (xy 63.5 114.3)
+		)
+		(stroke
+			(width 0)
+			(type default)
+		)
+	)
+	(wire
+		(pts
+			(xy 54.61 119.38) (xy 60.96 119.38)
+		)
+		(stroke
+			(width 0)
+			(type default)
+		)
+	)
 	(global_label "PWM5"
 		(shape input)
@@
 		)
 	)
+	(global_label "PWM1"
+		(shape input)
+		(at 42.926 94.742 0)
+		(fields_autoplaced yes)
+		(effects
+			(font
+				(size 1.27 1.27)
+			)
+			(justify left)
+		)
+		(property "Intersheetrefs" "${INTERSHEET_REFS}"
+			(at 51.2935 94.742 0)
+			(effects
+				(font
+					(size 1.27 1.27)
+				)
+				(justify left)
+				(hide yes)
+			)
+		)
+	)
 	(global_label "GndPlaca"
 		(shape input)
@@
 		)
 	)
-	(global_label "PWM1"
+	(global_label "GndPlaca"
 		(shape input)
-		(at 42.926 94.742 0)
+		(at 112.268 66.294 0)
 		(fields_autoplaced yes)
 		(effects
@@
 		)
 		(property "Intersheetrefs" "${INTERSHEET_REFS}"
-			(at 51.2935 94.742 0)
+			(at 124.143 66.294 0)
 			(effects
 				(font
@@
 		)
 	)
-	(global_label "GndPlaca"
+	(global_label "PWM4"
 		(shape input)
-		(at 112.268 66.294 0)
+		(at 131.826 55.88 180)
 		(fields_autoplaced yes)
 		(effects
@@
 				(size 1.27 1.27)
 			)
-			(justify left)
+			(justify right)
 		)
 		(property "Intersheetrefs" "${INTERSHEET_REFS}"
-			(at 124.143 66.294 0)
-			(effects
-				(font
-					(size 1.27 1.27)
-				)
-				(justify left)
-				(hide yes)
-			)
-		)
-	)
-	(global_label "PWM4"
+			(at 123.4585 55.88 0)
+			(effects
+				(font
+					(size 1.27 1.27)
+				)
+				(justify right)
+				(hide yes)
+			)
+		)
+	)
+	(global_label "PWM6"
 		(shape input)
-		(at 131.826 55.88 180)
+		(at 129.794 94.234 180)
 		(fields_autoplaced yes)
 		(effects
@@
 		)
 		(property "Intersheetrefs" "${INTERSHEET_REFS}"
-			(at 123.4585 55.88 0)
+			(at 121.4265 94.234 0)
 			(effects
 				(font
@@
 		)
 	)
-	(global_label "PWM6"
+	(global_label "PWM4"
 		(shape input)
-		(at 129.794 94.234 180)
+		(at 74.168 96.774 180)
 		(fields_autoplaced yes)
 		(effects
@@
 		)
 		(property "Intersheetrefs" "${INTERSHEET_REFS}"
-			(at 121.4265 94.234 0)
+			(at 65.8005 96.774 0)
 			(effects
 				(font
@@
 		)
 	)
-	(global_label "PWM4"
+	(global_label "PWM1"
 		(shape input)
-		(at 74.168 96.774 180)
+		(at 74.168 104.394 180)
 		(fields_autoplaced yes)
 		(effects
@@
 		)
 		(property "Intersheetrefs" "${INTERSHEET_REFS}"
-			(at 65.8005 96.774 0)
+			(at 65.8005 104.394 0)
 			(effects
 				(font
@@
 		)
 	)
-	(global_label "PWM1"
+	(global_label "VccPlaca"
 		(shape input)
-		(at 74.168 104.394 180)
+		(at 106.172 119.126 180)
 		(fields_autoplaced yes)
 		(effects
@@
 		)
 		(property "Intersheetrefs" "${INTERSHEET_REFS}"
-			(at 65.8005 104.394 0)
-			(effects
-				(font
-					(size 1.27 1.27)
-				)
-				(justify right)
-				(hide yes)
-			)
-		)
-	)
-	(global_label "VccPlaca"
-		(shape input)
-		(at 106.172 119.126 180)
-		(fields_autoplaced yes)
-		(effects
-			(font
-				(size 1.27 1.27)
-			)
-			(justify right)
-		)
-		(property "Intersheetrefs" "${INTERSHEET_REFS}"
 			(at 94.5992 119.126 0)
 			(effects
@@
 		(dnp no)
 		(fields_autoplaced yes)
-		(property "Reference" "M?"
+		(property "Reference" "M6"
 			(at 150.114 71.4485 0)
 			(effects
@@
 			(project "PCB"
 				(path "/ce73cf4f-b420-4ae1-b14f-64aecd900239"
-					(reference "M?")
+					(reference "M6")
 					(unit 1)
 				)
@@
 	(symbol
 		(lib_id "power:GND")
-		(at 59.436 119.126 0)
+		(at 60.96 119.38 0)
 		(unit 1)
 		(exclude_from_sim no)
@@
 		(fields_autoplaced yes)
 		(property "Reference" "#PWR09"
-			(at 59.436 125.476 0)
+			(at 60.96 125.73 0)
 			(effects
 				(font
@@
 		)
 		(property "Value" "GND"
-			(at 59.436 124.206 0)
+			(at 60.96 124.46 0)
 			(effects
 				(font
@@
 		)
 		(property "Footprint" ""
-			(at 59.436 119.126 0)
+			(at 60.96 119.38 0)
 			(effects
 				(font
@@
 		)
 		(property "Datasheet" ""
-			(at 59.436 119.126 0)
+			(at 60.96 119.38 0)
 			(effects
 				(font
@@
 		)
 		(property "Description" "Power symbol creates a global label with name \"GND\" , ground"
-			(at 59.436 119.126 0)
+			(at 60.96 119.38 0)
 			(effects
 				(font
@@
 		(dnp no)
 		(fields_autoplaced yes)
-		(property "Reference" "U?"
+		(property "Reference" "U2"
 			(at 114.808 114.554 0)
 			(effects
@@
 			)
 		)
-		(property "Footprint" ""
+		(property "Footprint" "Stepdown:Step down lm"
 			(at 108.458 120.142 0)
 			(effects
@@
 			(project "PCB"
 				(path "/ce73cf4f-b420-4ae1-b14f-64aecd900239"
-					(reference "U?")
+					(reference "U2")
 					(unit 1)
 				)
@@
 		(dnp no)
 		(fields_autoplaced yes)
-		(property "Reference" "U?"
+		(property "Reference" "U1"
 			(at 93.218 52.07 0)
 			(effects
@@
 			)
 		)
-		(property "Footprint" ""
+		(property "Footprint" "DOIT_ESP32:DOIT_ESP32_Devkit_mirko"
 			(at 79.248 58.674 0)
 			(effects
@@
 			(project "PCB"
 				(path "/ce73cf4f-b420-4ae1-b14f-64aecd900239"
-					(reference "U?")
+					(reference "U1")
 					(unit 1)
 				)
@@
 		(dnp no)
 		(fields_autoplaced yes)
-		(property "Reference" "M?"
+		(property "Reference" "M3"
 			(at 34.0471 83.566 0)
 			(effects
@@
 			(project "PCB"
 				(path "/ce73cf4f-b420-4ae1-b14f-64aecd900239"
-					(reference "M?")
+					(reference "M3")
 					(unit 1)
 				)
@@
 		(dnp no)
 		(fields_autoplaced yes)
-		(property "Reference" "M?"
+		(property "Reference" "M2"
 			(at 32.5231 68.326 0)
 			(effects
@@
 			(project "PCB"
 				(path "/ce73cf4f-b420-4ae1-b14f-64aecd900239"
-					(reference "M?")
+					(reference "M2")
 					(unit 1)
 				)
@@
 		(dnp no)
 		(fields_autoplaced yes)
-		(property "Reference" "M?"
+		(property "Reference" "M1"
 			(at 32.2691 53.34 0)
 			(effects
@@
 			(project "PCB"
 				(path "/ce73cf4f-b420-4ae1-b14f-64aecd900239"
-					(reference "M?")
+					(reference "M1")
 					(unit 1)
 				)
@@
 	(symbol
 		(lib_id "power:+12V")
-		(at 59.436 114.046 0)
+		(at 63.5 114.3 0)
 		(unit 1)
 		(exclude_from_sim no)
@@
 		(fields_autoplaced yes)
 		(property "Reference" "#PWR01"
-			(at 59.436 117.856 0)
+			(at 63.5 118.11 0)
 			(effects
 				(font
@@
 		)
 		(property "Value" "+12V"
-			(at 59.436 108.966 0)
+			(at 63.5 109.22 0)
 			(effects
 				(font
@@
 		)
 		(property "Footprint" ""
-			(at 59.436 114.046 0)
+			(at 63.5 114.3 0)
 			(effects
 				(font
@@
 		)
 		(property "Datasheet" ""
-			(at 59.436 114.046 0)
+			(at 63.5 114.3 0)
 			(effects
 				(font
@@
 		)
 		(property "Description" "Power symbol creates a global label with name \"+12V\""
-			(at 59.436 114.046 0)
+			(at 63.5 114.3 0)
 			(effects
 				(font
@@
 	(symbol
 		(lib_id "Connector:Barrel_Jack_MountingPin")
-		(at 51.816 116.586 0)
-		(unit 1)
-		(exclude_from_sim no)
-		(in_bom yes)
-		(on_board yes)
-		(dnp no)
-		(fields_autoplaced yes)
-		(property "Reference" "J?"
-			(at 51.816 107.95 0)
+		(at 46.99 116.84 0)
+		(unit 1)
+		(exclude_from_sim no)
+		(in_bom yes)
+		(on_board yes)
+		(dnp no)
+		(fields_autoplaced yes)
+		(property "Reference" "J1"
+			(at 46.99 108.204 0)
 			(effects
 				(font
@@
 		)
 		(property "Value" "Barrel_Jack_MountingPin"
-			(at 51.816 110.49 0)
+			(at 46.99 110.744 0)
 			(effects
 				(font
@@
 		)
 		(property "Footprint" "Connector_BarrelJack:BarrelJack_CUI_PJ-102AH_Horizontal"
-			(at 53.086 117.602 0)
+			(at 48.26 117.856 0)
 			(effects
 				(font
@@
 		)
 		(property "Datasheet" "~"
-			(at 53.086 117.602 0)
+			(at 48.26 117.856 0)
 			(effects
 				(font
@@
 		)
 		(property "Description" "DC Barrel Jack with a mounting pin"
-			(at 51.816 116.586 0)
+			(at 46.99 116.84 0)
 			(effects
 				(font
@@
 			(project "PCB"
 				(path "/ce73cf4f-b420-4ae1-b14f-64aecd900239"
-					(reference "J?")
+					(reference "J1")
 					(unit 1)
 				)
@@
 		(dnp no)
 		(fields_autoplaced yes)
-		(property "Reference" "M?"
+		(property "Reference" "M5"
 			(at 148.082 56.7165 0)
 			(effects
@@
 			(project "PCB"
 				(path "/ce73cf4f-b420-4ae1-b14f-64aecd900239"
-					(reference "M?")
+					(reference "M5")
 					(unit 1)
 				)
@@
 		(dnp no)
 		(fields_autoplaced yes)
-		(property "Reference" "M?"
+		(property "Reference" "M4"
 			(at 146.05 95.0705 0)
 			(effects
@@
 			(project "PCB"
 				(path "/ce73cf4f-b420-4ae1-b14f-64aecd900239"
-					(reference "M?")
-					(unit 1)
-				)
+					(reference "M4")
+					(unit 1)
+				)
